Commit message: add readme, add camera link, most basic version of camera transformation

File: MOMA_project/src/tm_description/xacro/tm12s.urdf.xacro (robot description, xacro)
@@ -12,4 +12,10 @@
   <!-- you must modify 'macro.tm12s-nominal.urdf.xacro' to 'user_defined.urdf.xacro'  -->
   <xacro:include filename="$(find tm_description)/xacro/macro.tm12s-nominal.urdf.xacro" />
+  <link name="camera_link"> </link>
+  <joint name="camera_joint" type="fixed">
+      <parent link="flange"/>
+      <child link="camera_link"/>
+      <origin xyz="0 -0.1 0.02" rpy="0 -${pi/2} 0"/>
+  </joint>
   <!--  -->
   <xacro:tmr_gazebo ns="$(arg ns)" prefix="$(arg prefix)" />

Commit message: tune urdf for camera_link

File: MOMA_project/src/tm_description/xacro/tm12s.urdf.xacro (robot description, xacro)
@@ -16,5 +16,5 @@
       <parent link="flange"/>
       <child link="camera_link"/>
-      <origin xyz="0 -0.1 0.02" rpy="0 -${pi/2} 0"/>
+      <origin xyz="0 -0.1372 0.0345" rpy="0 -${pi/2} 0"/>
   </joint>
   <!--  -->

Commit message: fix camera_link orientation

File: MOMA_project/src/tm_description/xacro/tm12s.urdf.xacro (robot description, xacro)
@@ -16,5 +16,5 @@
       <parent link="flange"/>
       <child link="camera_link"/>
-      <origin xyz="0 -0.1372 0.0345" rpy="0 -${pi/2} 0"/>
+      <origin xyz="0 -0.1372 0.0345" rpy="${pi/2} -${pi/2} 0"/>
   </joint>
   <!--  -->

Commit message: fine tune camera_link displacement wrt. base

File: MOMA_project/src/tm_description/xacro/tm12s.urdf.xacro (robot description, xacro)
@@ -16,5 +16,5 @@
       <parent link="flange"/>
       <child link="camera_link"/>
-      <origin xyz="0 -0.1372 0.0345" rpy="${pi/2} -${pi/2} 0"/>
+      <origin xyz="0 -0.1032 0.0345" rpy="${pi/2} -${pi/2} 0"/>
   </joint>
   <!--  -->
